Commit message: Added visualizer launch file and fixed URDF

File: packages/puzzlebot_description/urdf/test.urdf (robot description, URDF)
Before this commit: robot puzzlebot, 5 links, 4 joints
Joints:
- joint caster_joint: type continuous -> fixed
- joint wheel_l_joint: origin xyz=0.052 0.095 -0.0025 rpy=0 0 0 -> xyz=0.052 0.095 -0.0025 rpy=0 0 1.57
- joint wheel_r_joint: origin xyz=0.052 -0.095 -0.0025 rpy=0 0 0 -> xyz=0.052 -0.095 -0.0025 rpy=0 0 1.57

Commit message: Addition of URDF visualizer and modified meshes to support origin as the shape origin

File: packages/puzzlebot_description/urdf/test.urdf (robot description, URDF)
Before this commit: robot puzzlebot, 5 links, 4 joints
Links:
- link base_footprint: geometry visual mesh filename=package://puzzlebot_description/meshes/MCR2_puzzlebot_jetso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 scale=1.0 1.0 1.0
- link caster_link: geometry visual mesh filename=package://puzzlebot_description/meshes/MCR2_caster_wheel.stl scale=1.0 1.0 1.0
- link wheel_l_link: geometry visual mesh filename=package://puzzlebot_description/meshes/MCR2_wheel.stl scale=1.0 1.0 1.0
- link wheel_r_link: geometry visual mesh filename=package://puzzlebot_description/meshes/MCR2_wheel.stl scale=1.0 1.0 1.0
Joints:
- joint caster_joint: origin xyz=-0.095 0 -0.03 rpy=0 0 0 -> xyz=0.175 0 -0.04 rpy=0 0 0
