Commit message: Gazebo simulation

File: packages/puzzlebot_description/urdf/puzzlebot.urdf (robot description, URDF)
Before this commit: robot simple_robot, 4 links, 3 joints
Joints:
- joint wheel_l_joint: child wheel_l_link -> wheel_r_link; origin xyz=0.0 -0.052 -0.095 rpy=0 0 -1.57 -> xyz=0.0 -0.052 0.095 rpy=0 0 1.57
- joint wheel_r_joint: child wheel_r_link -> wheel_l_link; origin xyz=0.0 -0.052 0.095 rpy=0 0 1.57 -> xyz=0.0 -0.052 -0.095 rpy=0 0 -1.57

Commit message: Addition of customized walls and lidar sensor to urdf

File: packages/puzzlebot_description/urdf/puzzlebot.urdf (robot description, URDF)
Before this commit: robot simple_robot, 4 links, 3 joints
Links:
- added link laser_frame
Joints:
- added joint laser_joint: type fixed, parent base_link, child laser_frame, origin xyz=0.122 0 0.212 rpy=0 0 0

Commit message: Modifications upon TFs and gazebo tags for lidar and velocity controller

File: packages/puzzlebot_description/urdf/puzzlebot.urdf (robot description, URDF)
Before this commit: robot simple_robot, 5 links, 4 joints
Links:
- removed link laser_frame
- added link base_footprint, mass 0.001; collision mesh filename=file://$(find puzzlebot_description)/meshes/MCR2_puzzlebot_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 scale=1.0 1.0 1.0; visual mesh filename=file://$(find puzzlebot_description)/meshes/MCR2_puzzlebot_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 scale=1.0 1.0 1.0
- added link laser_link
- link base_link: geometry collision box size=0.0 0.0 0.0; visual box size=0.0 0.0 0.0
Joints:
- added joint base_link_joint: type fixed, parent base_footprint, child base_link, origin xyz=0 0 0.05 rpy=0 0 0
- joint caster_joint: axis 0 0 1 -> (none); origin xyz=0.15 -0.095 0 rpy=-1.57 0 0 -> xyz=0.175 0 -0.04 rpy=0 0 0
- joint laser_joint: child laser_frame -> laser_link; origin xyz=0.122 0 0.212 rpy=0 0 0 -> xyz=0.05 0 0.11 rpy=0 0 0
- joint wheel_l_joint: axis 0 0 1 -> -1 0 0; child wheel_r_link -> wheel_l_link; origin xyz=0.0 -0.052 0.095 rpy=0 0 1.57 -> xyz=0.052 0.095 -0.0025 rpy=0 0 1.57
- joint wheel_r_joint: axis 0 0 1 -> -1 0 0; child wheel_l_link -> wheel_r_link; origin xyz=0.0 -0.052 -0.095 rpy=0 0 -1.57 -> xyz=0.052 -0.095 -0.0025 rpy=0 0 1.57

Commit message: Improvements over puzzlebot physics, it works better with small velocities

File: packages/puzzlebot_description/urdf/puzzlebot.urdf (robot description, URDF)
Before this commit: robot simple_robot, 6 links, 5 joints
Links:
- link base_footprint: mass 0.001 -> 10.5
- link base_link: mass 0.001 -> None
- link caster_link: mass 0.5 -> 3.5
- link wheel_l_link: mass 0.5 -> 0.3
- link wheel_r_link: mass 0.5 -> 0.3

Commit message: Fixed odom transform

File: packages/puzzlebot_description/urdf/puzzlebot.urdf (robot description, URDF)
Before this commit: robot simple_robot, 6 links, 5 joints
Links:
- added link odom
Joints:
- added joint odom_joint: type fixed, parent odom, child base_footprint, origin xyz=0 0 0 rpy=0 0 0

Commit message: Addition of necessary config files to run slam_toolbox

File: packages/puzzlebot_description/urdf/puzzlebot.urdf (robot description, URDF)
Before this commit: robot simple_robot, 7 links, 6 joints
Links:
- removed link laser_link
- added link laser_frame
Joints:
- joint laser_joint: child laser_link -> laser_frame

Commit message: Robot simulation now is compatible with navstack 2

File: packages/puzzlebot_description/urdf/puzzlebot.urdf (robot description, URDF)
Before this commit: robot simple_robot, 7 links, 6 joints
Joints:
- joint caster_joint: origin xyz=0.175 0 -0.04 rpy=0 0 0 -> xyz=-0.175 0 -0.0425 rpy=0 0 0
- joint wheel_l_joint: axis -1 0 0 -> 1 0 0
- joint wheel_r_joint: axis -1 0 0 -> 1 0 0

Commit message: Fixed caster wheel transform

File: packages/puzzlebot_description/urdf/puzzlebot.urdf (robot description, URDF)
Before this commit: robot simple_robot, 7 links, 6 joints
Joints:
- joint caster_joint: origin xyz=-0.175 0 -0.0425 rpy=0 0 0 -> xyz=-0.075 0 -0.0425 rpy=0 0 0
