Commit message: Deleted redundant launchfiles and urdf files

File: packages/puzzlebot_description/urdf/gazebo_tags.xacro (robot description, xacro)
@@ -4,4 +4,10 @@
     <!-- Conditionally include ros2_control configuration and diff_drive plugin -->
     <xacro:if value="${use_gazebo_controllers}">
+      <link name="odom"/>
+      <joint name="odom_joint" type="fixed">
+        <parent link="odom"/>
+        <child link="base_footprint"/>
+        <origin xyz="0 0 0" rpy="0 0 0"/>
+      </joint>
       <!-- ros2_control Configuration -->
       <ros2_control name="GazeboSystem" type="system">

File: packages/puzzlebot_description/urdf/robot.xacro (robot description, xacro)
@@ -2,8 +2,13 @@
 <robot name="puzzlebot"
   xmlns:xacro="http://ros.org/wiki/xacro">
-  <!-- Include the puzzlebot modular description -->
+  <!-- Declare arguments -->
+  <xacro:arg name="prefix" default=""/>
+  <xacro:arg name="use_gazebo" default="true"/>
+  <xacro:arg name="use_gazebo_controllers" default="true"/>
+  <!-- Include macros -->
   <xacro:include filename="$(find puzzlebot_description)/urdf/puzzlebot.xacro"/>
   <xacro:include filename="$(find puzzlebot_description)/urdf/gazebo_tags.xacro"/>
-  <!-- Instantiate the macro with optional prefix -->
-  <xacro:puzzlebot_description prefix=""/>
+  <!-- Call macros with args -->
+  <xacro:puzzlebot_description prefix="$(arg prefix)"/>
+  <xacro:gazebo_tags use_gazebo_controllers="$(arg use_gazebo_controllers)"/>
 </robot>

Commit message: Now the wheels are blue

File: packages/puzzlebot_description/urdf/gazebo_tags.xacro (robot description, xacro)
@@ -88,4 +88,10 @@
       <material>Gazebo/Black</material>
     </gazebo>
+    <gazebo reference="wheel_l_link">
+      <material>Gazebo/Blue</material>
+    </gazebo>
+    <gazebo reference="wheel_r_link">
+      <material>Gazebo/Blue</material>
+    </gazebo>
   </xacro:macro>
 </robot>

Commit message: MCL working with Gazebo and ROS2

File: packages/puzzlebot_description/urdf/gazebo_tags.xacro (robot description, xacro)
@@ -1,13 +1,16 @@
 <?xml version="1.0"?>
 <robot xmlns:xacro="http://ros.org/wiki/xacro">
-  <xacro:macro name="gazebo_tags" params="use_gazebo_controllers:=false">
+  <xacro:macro name="gazebo_tags" params="use_gazebo_controllers:=false use_gazebo_odom:=false">
     <!-- Conditionally include ros2_control configuration and diff_drive plugin -->
     <xacro:if value="${use_gazebo_controllers}">
-      <link name="odom"/>
-      <joint name="odom_joint" type="fixed">
-        <parent link="odom"/>
-        <child link="base_footprint"/>
-        <origin xyz="0 0 0" rpy="0 0 0"/>
-      </joint>
+      <xacro:if value="${use_gazebo_odom}">
+        <xacro:property name="odom_frame" value="odom"/>
+        <link name="odom"/>
+        <joint name="odom_joint" type="fixed">
+          <parent link="odom"/>
+          <child link="base_footprint"/>
+          <origin xyz="0 0 0" rpy="0 0 0"/>
+        </joint>
+      </xacro:if>
       <!-- ros2_control Configuration -->
       <ros2_control name="GazeboSystem" type="system">
@@ -43,6 +46,6 @@
           <odometry_frame>odom</odometry_frame>
           <robot_base_frame>base_footprint</robot_base_frame>
-          <publish_odom>true</publish_odom>
-          <publish_odom_tf>true</publish_odom_tf>
+          <publish_odom>false</publish_odom>
+          <publish_odom_tf>false</publish_odom_tf>
           <publish_wheel_tf>false</publish_wheel_tf>
         </plugin>
@@ -50,10 +53,10 @@
     </xacro:if>
     <!-- Joint State Publisher is always included (or make this conditional instead if needed) -->
-    <gazebo>
+    <!-- <gazebo>
       <plugin name="gazebo_ros_joint_state_publisher" filename="libgazebo_ros_joint_state_publisher.so">
         <joint_name>wheel_l_joint</joint_name>
         <joint_name>wheel_r_joint</joint_name>
       </plugin>
-    </gazebo>
+    </gazebo> -->
     <!-- Gazebo Sensor: Laser -->
     <gazebo reference="laser_frame">

File: packages/puzzlebot_description/urdf/robot.xacro (robot description, xacro)
@@ -6,4 +6,5 @@
   <xacro:arg name="use_gazebo" default="true"/>
   <xacro:arg name="use_gazebo_controllers" default="true"/>
+  <xacro:arg name="use_gazebo_odom" default="false"/>
   <!-- Include macros -->
   <xacro:include filename="$(find puzzlebot_description)/urdf/puzzlebot.xacro"/>

Commit message: Added parameter to use or not gazebo odometry

File: packages/puzzlebot_description/urdf/gazebo_tags.xacro (robot description, xacro)
@@ -4,35 +4,11 @@
     <!-- Conditionally include ros2_control configuration and diff_drive plugin -->
     <xacro:if value="${use_gazebo_controllers}">
-      <xacro:if value="${use_gazebo_odom}">
-        <xacro:property name="odom_frame" value="odom"/>
-        <link name="odom"/>
-        <joint name="odom_joint" type="fixed">
-          <parent link="odom"/>
-          <child link="base_footprint"/>
-          <origin xyz="0 0 0" rpy="0 0 0"/>
-        </joint>
-      </xacro:if>
-      <!-- ros2_control Configuration -->
-      <ros2_control name="GazeboSystem" type="system">
-        <hardware>
-          <plugin>gazebo_ros2_control/GazeboSystem</plugin>
-        </hardware>
-        <!-- Joint Configuration -->
-        <joint name="wheel_l_joint">
-          <command_interface name="velocity"/>
-          <state_interface name="velocity"/>
-        </joint>
-        <joint name="wheel_r_joint">
-          <command_interface name="velocity"/>
-          <state_interface name="velocity"/>
-        </joint>
-      </ros2_control>
       <!-- Gazebo Plugin: Differential Drive -->
       <gazebo>
         <plugin name="diff_drive" filename="libgazebo_ros_diff_drive.so">
           <ros>
-            <remapping>odom:=/puzzlebot_odom</remapping>
+            <remapping>odom:=/odom</remapping>
           </ros>
-          <!-- Wheel Information -->
+          <!-- Wheel Info -->
           <left_joint>wheel_l_joint</left_joint>
           <right_joint>wheel_r_joint</right_joint>
@@ -43,21 +19,14 @@
           <max_wheel_torque>109</max_wheel_torque>
           <max_wheel_acceleration>5.0</max_wheel_acceleration>
-          <!-- Output -->
+          <!-- Output config based on odom flag -->
           <odometry_frame>odom</odometry_frame>
           <robot_base_frame>base_footprint</robot_base_frame>
-          <publish_odom>false</publish_odom>
-          <publish_odom_tf>false</publish_odom_tf>
+          <publish_odom><xacro:if value="${use_gazebo_odom}">true</xacro:if><xacro:unless value="${use_gazebo_odom}">false</xacro:unless></publish_odom>
+          <publish_odom_tf><xacro:if value="${use_gazebo_odom}">true</xacro:if><xacro:unless value="${use_gazebo_odom}">false</xacro:unless></publish_odom_tf>
           <publish_wheel_tf>false</publish_wheel_tf>
         </plugin>
       </gazebo>
     </xacro:if>
-    <!-- Joint State Publisher is always included (or make this conditional instead if needed) -->
-    <!-- <gazebo>
-      <plugin name="gazebo_ros_joint_state_publisher" filename="libgazebo_ros_joint_state_publisher.so">
-        <joint_name>wheel_l_joint</joint_name>
-        <joint_name>wheel_r_joint</joint_name>
-      </plugin>
-    </gazebo> -->
-    <!-- Gazebo Sensor: Laser -->
+    <!-- Laser sensor -->
     <gazebo reference="laser_frame">
       <sensor name="laser" type="ray">
@@ -87,5 +56,5 @@
       </sensor>
     </gazebo>
-    <!-- Gazebo Material: Base Footprint -->
+    <!-- Materials -->
     <gazebo reference="base_footprint">
       <material>Gazebo/Black</material>

File: packages/puzzlebot_description/urdf/robot.xacro (robot description, xacro)
@@ -12,4 +12,6 @@
   <!-- Call macros with args -->
   <xacro:puzzlebot_description prefix="$(arg prefix)"/>
-  <xacro:gazebo_tags use_gazebo_controllers="$(arg use_gazebo_controllers)"/>
+  <xacro:gazebo_tags
+      use_gazebo_controllers="$(arg use_gazebo_controllers)"
+      use_gazebo_odom="$(arg use_gazebo_odom)"/>
 </robot>
