Commit message: Functioning launch file for real puzzlebot

File: packages/puzzlebot_description/urdf/puzzlebot.xacro (robot description, xacro)
@@ -96,4 +96,5 @@
     </link>
     <link name="${prefix}laser_frame"/>
+    <link name="laser"/>
     <!-- Joints -->
     <joint name="${prefix}base_link_joint" type="fixed">
@@ -124,4 +125,9 @@
       <origin xyz="0.05 0 0.11" rpy="0 0 0"/>
     </joint>
+   <joint name="laser_frame_to_laser" type="fixed">
+    <parent link="laser_frame"/>
+    <child link="laser"/>
+    <origin xyz="0 0 0" rpy="0 0 3.14"/>
+   </joint>
   </xacro:macro>
 </robot>

Commit message: testing tf_saver

File: packages/puzzlebot_description/urdf/puzzlebot.xacro (robot description, xacro)
@@ -95,4 +95,5 @@
       </inertial>
     </link>
+    <link name="${prefix}camera_base_link"/>
     <link name="${prefix}laser_frame"/>
     <link name="laser"/>
@@ -120,4 +121,9 @@
       <origin xyz="-0.075 0 -0.0425" rpy="0 0 0"/>
     </joint>
+    <joint name="${prefix}camera_base_joint" type="fixed">
+        <parent link="${prefix}base_link"/>
+        <child link="${prefix}camera_base_link"/>
+        <origin xyz="0.112 0 0.065" rpy="0 0 0"/>
+    </joint>
     <joint name="${prefix}laser_joint" type="fixed">
       <parent link="${prefix}base_link"/>

Commit message: Working aruco tf saver

File: packages/puzzlebot_description/urdf/puzzlebot.xacro (robot description, xacro)
@@ -124,5 +124,5 @@
         <parent link="${prefix}base_link"/>
         <child link="${prefix}camera_base_link"/>
-        <origin xyz="0.112 0 0.065" rpy="0 0 0"/>
+        <origin xyz="0.112 0 0.065" rpy="-1.57 0 -1.57"/>
     </joint>
     <joint name="${prefix}laser_joint" type="fixed">
