Commit message: Puzzlebot in a small world simulation

File: packages/puzzlebot_description/urdf/boxes.xacro (robot description, xacro)
@@ -2,6 +2,6 @@
 <robot xmlns:xacro="http://ros.org/wiki/xacro" name="simple_rectangle">
   <!-- Rectangle dimensions -->
-  <xacro:property name="length" value="0.5"/>  <!-- x-axis -->
-  <xacro:property name="width" value="0.3"/>   <!-- y-axis -->
+  <xacro:property name="length" value="0.3"/>  <!-- x-axis -->
+  <xacro:property name="width" value="0.2"/>   <!-- y-axis -->
   <xacro:property name="height" value="0.2"/>  <!-- z-axis -->
   <xacro:property name="box_mass" value="1.0"/>
